File: 2x2x4/build/2x2x4-LED-Panel.kicad_sch (KiCad schematic)
At the start: 2 parts

Commit message: Added test points
Parts:
- added TP1: TestPoint, Schrune:TestPoint_Pad_1.0x1.0mm, symbol TestPoint
- added TP2: TestPoint, Schrune:TestPoint_Pad_1.5x1.5mm, symbol TestPoint
- added TP3, TP4: TestPoint, Schrune:TestPoint_Pad_D1.0mm, symbol TestPoint
Connections:
- net GND: now also TP2.1
- net V+: now also TP1.1
- net pwm_cool: now also TP3.1
- net pwm_warm: now also TP4.1

Commit message: 2x2x4 finishing touches
Parts:
- TP1, TP2, TP3, TP4: now not fitted; now left out of the parts list
Changed lines of the file:
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@@
 		(body_style 1)
 		(exclude_from_sim no)
-		(in_bom yes)
-		(on_board yes)
-		(in_pos_files yes)
-		(dnp no)
+		(in_bom no)
+		(on_board yes)
+		(in_pos_files yes)
+		(dnp yes)
 		(property "Reference" "TP1"
 			(at 76.2 172.72 0)
@@
 		(body_style 1)
 		(exclude_from_sim no)
-		(in_bom yes)
-		(on_board yes)
-		(in_pos_files yes)
-		(dnp no)
+		(in_bom no)
+		(on_board yes)
+		(in_pos_files yes)
+		(dnp yes)
 		(property "Reference" "TP4"
 			(at 482.6 96.52 0)
@@
 		(body_style 1)
 		(exclude_from_sim no)
-		(in_bom yes)
-		(on_board yes)
-		(in_pos_files yes)
-		(dnp no)
+		(in_bom no)
+		(on_board yes)
+		(in_pos_files yes)
+		(dnp yes)
 		(property "Reference" "TP3"
 			(at 685.8 96.52 0)
@@
 		(body_style 1)
 		(exclude_from_sim no)
-		(in_bom yes)
-		(on_board yes)
-		(in_pos_files yes)
-		(dnp no)
+		(in_bom no)
+		(on_board yes)
+		(in_pos_files yes)
+		(dnp yes)
 		(property "Reference" "TP2"
 			(at 279.4 172.72 0)
