File: 2x2x4/build/2x2x4-LED-Panel.kicad_pcb (KiCad board)
At the start: 2 copper layers, 75 x 30 mm, 58 parts, among them U1 PT4115, U2 PT4115, U3 PT4115, U4 PT4115

Commit message: Added test points
Parts:
- added TP+: TestPoint, Schrune:TestPoint_Pad_1.0x1.0mm, F.Cu at (169.8, 107.2)
- added TP-: TestPoint, Schrune:TestPoint_Pad_1.5x1.5mm, F.Cu at (172.2, 124.0)
- added TP_C: TestPoint, Schrune:TestPoint_Pad_D1.0mm, F.Cu at (128.8, 115.2)
- added TP_W: TestPoint, Schrune:TestPoint_Pad_D1.0mm, F.Cu at (122.2, 114.0)
Routing:
- net V+: track 33.1 -> 35.8 mm, vias 5 -> 6

Commit message: 2x2x4 finishing touches
Parts:
- moved TP1 1.42 mm to (168.4, 106.8)
- renumbered TP+ to TP1, TP- to TP2, TP_C to TP3, TP_W to TP4
Routing:
- net V+: track 35.8 -> 36.8 mm
Other:
- board text added: "- +"
- board text added: "TP+"
- board text added: "TP-"
- board text added: "TP_C"
- board text added: "TP_W"

Commit message: Build changes
Other:
- board text added: "2x2x4 LED Panel v2.0.0 - July 2026"
