File: hex-connector-advanced/build/Hex Connector - Advanced.kicad_sch (KiCad schematic)
At the start: 8 parts

Commit message: Finished up HCA
Parts:
- removed DC1: KLDVX-0202-B, Schrune:KLDVX_0202_B, symbol KLDVX-0202-B
- added DC1: LDC-121-L-051-1AG-09, Schrune:LDC_121_L_051_1AG_09, symbol LDC-121-L-051-1AG-09
Connections:
- net GND: now also DC1.2, DC1.3
- net V+: now also DC1.1
Changed lines of the file:
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@@
     )
   )
-  (symbol (lib_id "KLDVX-0202-B") (at 685.80 177.80 0) (unit 1)
+  (symbol (lib_id "LDC-121-L-051-1AG-09") (at 685.80 177.80 0) (unit 1)
     (in_bom yes) (on_board yes) (dnp no)
     (property "Reference" "DC1" (at 685.80 172.72 0)
       (effects (font (size 1.27 1.27)))
     )
-    (property "Value" "KLDVX-0202-B" (at 685.80 182.88 0)
+    (property "Value" "LDC-121-L-051-1AG-09" (at 685.80 182.88 0)
       (effects (font (size 1.27 1.27)))
     )
-    (property "Footprint" "Schrune:KLDVX_0202_B" (at 685.80 185.42 0) (hide yes)
+    (property "Footprint" "Schrune:LDC_121_L_051_1AG_09" (at 685.80 185.42 0) (hide yes)
       (effects (font (size 1.27 1.27)))
     )
