File: hex-connector-advanced/build/Hex Connector - Advanced.kicad_pcb (KiCad board)
At the start: 2 copper layers, 60 x 52 mm, 8 parts

Commit message: Finished up HCA
Parts:
- removed DC 15v-24v: KLDVX-0202-B, Schrune:KLDVX_0202_B
- removed MCU: PZ2.54-2X5P-H25, Schrune:PZ2_54_2X5P_H25
- added DC1: LDC-121-L-051-1AG-09, Schrune:LDC_121_L_051_1AG_09, F.Cu at (110.2, 126.1)
- added H7: PZ2.54-2X5P-H25, Schrune:PZ2_54_2X5P_H25, F.Cu at (115.0, 113.7)
Other:
- board text added: "Hex LP Connector Advanced v1.0.0 - July 2026"

Commit message: Added mounting holes to hex connectors
Parts:
- 15-30V DC: renamed from DC1
Other:
- outline, holes or cut-outs redrawn
- board text added: "Hex LP Connector Advanced v1.0.2 - July 2026"
- board text removed: "Hex LP Connector Advanced v1.0.0 - July 2026"
Changed lines of the file:
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@@
 			(drillshape 0)
 			(scaleselection 1)
-			(outputdirectory "gerber/")
+			(outputdirectory "../../hex-connector-simple/build/gerbers/")
 		)
 	)
@@
 		(layer "F.Cu")
 		(at 110.2375 126.1125)
-		(property "Reference" "DC1"
+		(property "Reference" "15-30V DC"
 			(at 4.5 -5.5 0)
 			(layer "F.SilkS")
@@
 	)
 	(gr_line
-		(start 100.528358 101.06875)
+		(start 100.5 101)
 		(end 86.056717 126.134375)
 		(stroke
@@
 	)
 	(gr_line
-		(start 129.471642 101.06875)
-		(end 100.528358 101.06875)
-		(stroke
-			(width 0.337672)
-			(type solid)
-		)
-		(layer "F.Cu")
-		(net "/pwm_warm")
-	)
-	(gr_line
 		(start 129.471642 151.2)
 		(end 143.943283 126.134375)
@@
 	(gr_line
 		(start 143.943283 126.134375)
-		(end 129.471642 101.06875)
+		(end 136.75 113.5)
 		(stroke
 			(width 0.337672)
@@
 		(layer "Edge.Cuts")
 	)
+	(gr_circle
+		(center 89 126)
+		(end 90.25 126)
+		(stroke
+			(width 0.05)
+			(type solid)
+		)
+		(fill no)
+		(layer "Edge.Cuts")
+	)
 	(gr_line
 		(start 100 100)
@@
 	)
 	(gr_circle
+		(center 102 103)
+		(end 103.25 103)
+		(stroke
+			(width 0.05)
+			(type solid)
+		)
+		(fill no)
+		(layer "Edge.Cuts")
+	)
+	(gr_circle
+		(center 102 148)
+		(end 103.25 148)
+		(stroke
+			(width 0.05)
+			(type solid)
+		)
+		(fill no)
+		(layer "Edge.Cuts")
+	)
+	(gr_circle
 		(center 107 140)
 		(end 111.5 140)
@@
 		(layer "Edge.Cuts")
 	)
+	(gr_circle
+		(center 128 103)
+		(end 129.25 103)
+		(stroke
+			(width 0.05)
+			(type solid)
+		)
+		(fill no)
+		(layer "Edge.Cuts")
+	)
+	(gr_circle
+		(center 128 148)
+		(end 129.25 148)
+		(stroke
+			(width 0.05)
+			(type solid)
+		)
+		(fill no)
+		(layer "Edge.Cuts")
+	)
 	(gr_line
 		(start 130 100)
@@
 		(layer "Edge.Cuts")
 	)
+	(gr_circle
+		(center 141 126)
+		(end 142.25 126)
+		(stroke
+			(width 0.05)
+			(type solid)
+		)
+		(fill no)
+		(layer "Edge.Cuts")
+	)
 	(gr_line
 		(start 145 125.980762)
@@
 		)
 	)
-	(gr_text "Hex LP Connector Advanced\nv1.0.0 - July 2026"
-		(at 141.25 128.5 0)
+	(gr_text "Hex LP Connector Advanced\nv1.0.2 - July 2026"
+		(at 139.3 128.3 0)
 		(layer "B.SilkS")
 		(effects
@@
 	)
 	(segment
-		(start 135.645 114.355)
-		(end 136.5 113.5)
+		(start 94.936148 114.355)
+		(end 94.936148 110.963852)
 		(width 0.254)
 		(layer "F.Cu")
@@
 	)
 	(segment
-		(start 94.936148 114.355)
-		(end 94.936148 110.963852)
-		(width 0.254)
+		(start 113.27 101)
+		(end 100.5 101)
+		(width 0.2)
 		(layer "F.Cu")
 		(net "/pwm_warm")
@@
 	)
 	(segment
-		(start 113.33875 101.06875)
-		(end 100.528358 101.06875)
+		(start 135.135852 137.606)
+		(end 136.1 138.570148)
 		(width 0.254)
 		(layer "F.Cu")
@@
 	)
 	(segment
-		(start 135.135852 137.606)
-		(end 136.1 138.570148)
-		(width 0.254)
+		(start 115 102.73)
+		(end 113.27 101)
+		(width 0.2)
 		(layer "F.Cu")
 		(net "/pwm_warm")
@@
 	)
 	(segment
-		(start 135.135852 114.355)
-		(end 135.645 114.355)
+		(start 136.1 138.570148)
+		(end 136.1 139.7)
 		(width 0.254)
 		(layer "F.Cu")
@@
 	)
 	(segment
-		(start 136.1 138.570148)
-		(end 136.1 139.7)
+		(start 98.9 104)
+		(end 98.8 104.1)
 		(width 0.254)
 		(layer "F.Cu")
@@
 	)
 	(segment
-		(start 115 102.73)
-		(end 113.33875 101.06875)
+		(start 135.895 114.355)
+		(end 136.75 113.5)
+		(width 0.254)
+		(layer "F.Cu")
+		(net "/pwm_warm")
+	)
+	(segment
+		(start 135.135852 114.355)
+		(end 135.895 114.355)
 		(width 0.254)
 		(layer "F.Cu")
