File: hex-connector-simple/build/Hex Connector - Simple.kicad_pcb (KiCad board)
At the start: 2 copper layers, 60 x 52 mm, 6 parts

Commit message: Added mounting holes to hex connectors
Other:
- outline, holes or cut-outs redrawn
- board text added: "+ -"
- board text added: "Hex LP Connector v1.0.0 - July 2026"
